Commit message: auto: update 2026-04-30 01:43:54

File: turtlebot3_manipulation/turtlebot3_manipulation_description/xacro/turtlebot3_manipulation.urdf.xacro (robot description, xacro)
@@ -6,4 +6,7 @@
   <xacro:arg name="fake_sensor_commands" default="false" />
   <xacro:arg name="use_camera_driver_tf" default="false" />
+  <xacro:arg name="use_eef_usb_camera" default="true" />
+  <xacro:arg name="eef_usb_camera_xyz" default="0.0 0.0 0.05" />
+  <xacro:arg name="eef_usb_camera_rpy" default="0.0 0.0 0.0" />
   <xacro:include filename="$(find turtlebot3_manipulation_description)/gazebo/materials.xacro" />
   <xacro:include filename="$(find turtlebot3_manipulation_description)/xacro/turtlebot3_waffle_pi.urdf.xacro" />
@@ -86,4 +89,39 @@
   <xacro:open_manipulator_x prefix="$(arg prefix)" />
   <xacro:open_manipulator_x_gazebo prefix="$(arg prefix)" />
+  <xacro:if value="$(arg use_eef_usb_camera)">
+    <joint name="$(arg prefix)eef_usb_camera_joint" type="fixed">
+      <parent link="$(arg prefix)end_effector_link"/>
+      <child link="$(arg prefix)eef_usb_camera_link"/>
+      <origin xyz="$(arg eef_usb_camera_xyz)" rpy="$(arg eef_usb_camera_rpy)"/>
+    </joint>
+    <link name="$(arg prefix)eef_usb_camera_link">
+      <visual>
+        <origin xyz="0.015 0 0" rpy="0 0 0"/>
+        <geometry>
+          <box size="0.03 0.03 0.02"/>
+        </geometry>
+        <material name="dark_grey">
+          <color rgba="0.1 0.1 0.1 1"/>
+        </material>
+      </visual>
+      <collision>
+        <origin xyz="0.015 0 0" rpy="0 0 0"/>
+        <geometry>
+          <box size="0.03 0.03 0.02"/>
+        </geometry>
+      </collision>
+      <inertial>
+        <origin xyz="0.015 0 0" rpy="0 0 0"/>
+        <mass value="0.02"/>
+        <inertia ixx="0.00001" ixy="0.0" ixz="0.0" iyy="0.00001" iyz="0.0" izz="0.00001"/>
+      </inertial>
+    </link>
+    <joint name="$(arg prefix)eef_usb_camera_optical_joint" type="fixed">
+      <parent link="$(arg prefix)eef_usb_camera_link"/>
+      <child link="$(arg prefix)eef_usb_camera_optical_frame"/>
+      <origin xyz="0 0 0" rpy="${-pi/2} 0 ${-pi/2}"/>
+    </joint>
+    <link name="$(arg prefix)eef_usb_camera_optical_frame"/>
+  </xacro:if>
   <xacro:turtlebot3_manipulation_system
     name="TurtleBot3ManipulationSystem" prefix="$(arg prefix)" use_sim="$(arg use_sim)"

Commit message: auto: update 2026-04-30 02:00:56

File: turtlebot3_manipulation/turtlebot3_manipulation_description/xacro/turtlebot3_manipulation.urdf.xacro (robot description, xacro)
@@ -7,5 +7,6 @@
   <xacro:arg name="use_camera_driver_tf" default="false" />
   <xacro:arg name="use_eef_usb_camera" default="true" />
-  <xacro:arg name="eef_usb_camera_xyz" default="0.0 0.0 0.05" />
+  <xacro:arg name="eef_usb_camera_parent" default="link5" />
+  <xacro:arg name="eef_usb_camera_xyz" default="0.06 0.0 0.10" />
   <xacro:arg name="eef_usb_camera_rpy" default="0.0 0.0 0.0" />
   <xacro:include filename="$(find turtlebot3_manipulation_description)/gazebo/materials.xacro" />
@@ -91,5 +92,5 @@
   <xacro:if value="$(arg use_eef_usb_camera)">
     <joint name="$(arg prefix)eef_usb_camera_joint" type="fixed">
-      <parent link="$(arg prefix)end_effector_link"/>
+      <parent link="$(arg prefix)$(arg eef_usb_camera_parent)"/>
       <child link="$(arg prefix)eef_usb_camera_link"/>
       <origin xyz="$(arg eef_usb_camera_xyz)" rpy="$(arg eef_usb_camera_rpy)"/>

Commit message: auto: update 2026-04-30 02:13:52

File: turtlebot3_manipulation/turtlebot3_manipulation_description/xacro/turtlebot3_manipulation.urdf.xacro (robot description, xacro)
@@ -7,6 +7,6 @@
   <xacro:arg name="use_camera_driver_tf" default="false" />
   <xacro:arg name="use_eef_usb_camera" default="true" />
-  <xacro:arg name="eef_usb_camera_parent" default="link5" />
-  <xacro:arg name="eef_usb_camera_xyz" default="0.06 0.0 0.10" />
+  <xacro:arg name="eef_usb_camera_parent" default="dummy_mimic_fix" />
+  <xacro:arg name="eef_usb_camera_xyz" default="0.0 0.0 0.04" />
   <xacro:arg name="eef_usb_camera_rpy" default="0.0 0.0 0.0" />
   <xacro:include filename="$(find turtlebot3_manipulation_description)/gazebo/materials.xacro" />
@@ -92,5 +92,5 @@
   <xacro:if value="$(arg use_eef_usb_camera)">
     <joint name="$(arg prefix)eef_usb_camera_joint" type="fixed">
-      <parent link="$(arg prefix)$(arg eef_usb_camera_parent)"/>
+      <parent link="$(arg eef_usb_camera_parent)"/>
       <child link="$(arg prefix)eef_usb_camera_link"/>
       <origin xyz="$(arg eef_usb_camera_xyz)" rpy="$(arg eef_usb_camera_rpy)"/>

Commit message: auto: update 2026-04-30 02:17:03

File: turtlebot3_manipulation/turtlebot3_manipulation_description/xacro/turtlebot3_manipulation.urdf.xacro (robot description, xacro)
@@ -8,5 +8,5 @@
   <xacro:arg name="use_eef_usb_camera" default="true" />
   <xacro:arg name="eef_usb_camera_parent" default="dummy_mimic_fix" />
-  <xacro:arg name="eef_usb_camera_xyz" default="0.0 0.0 0.04" />
+  <xacro:arg name="eef_usb_camera_xyz" default="0.0 0.0 0.065" />
   <xacro:arg name="eef_usb_camera_rpy" default="0.0 0.0 0.0" />
   <xacro:include filename="$(find turtlebot3_manipulation_description)/gazebo/materials.xacro" />
@@ -98,7 +98,7 @@
     <link name="$(arg prefix)eef_usb_camera_link">
       <visual>
-        <origin xyz="0.015 0 0" rpy="0 0 0"/>
+        <origin xyz="0.045 0 0" rpy="0 0 0"/>
         <geometry>
-          <box size="0.03 0.03 0.02"/>
+          <box size="0.09 0.05 0.045"/>
         </geometry>
         <material name="dark_grey">
@@ -107,11 +107,11 @@
       </visual>
       <collision>
-        <origin xyz="0.015 0 0" rpy="0 0 0"/>
+        <origin xyz="0.045 0 0" rpy="0 0 0"/>
         <geometry>
-          <box size="0.03 0.03 0.02"/>
+          <box size="0.09 0.05 0.045"/>
         </geometry>
       </collision>
       <inertial>
-        <origin xyz="0.015 0 0" rpy="0 0 0"/>
+        <origin xyz="0.045 0 0" rpy="0 0 0"/>
         <mass value="0.02"/>
         <inertia ixx="0.00001" ixy="0.0" ixz="0.0" iyy="0.00001" iyz="0.0" izz="0.00001"/>

Commit message: auto: update 2026-04-30 02:19:52

File: turtlebot3_manipulation/turtlebot3_manipulation_description/xacro/turtlebot3_manipulation.urdf.xacro (robot description, xacro)
@@ -98,7 +98,7 @@
     <link name="$(arg prefix)eef_usb_camera_link">
       <visual>
-        <origin xyz="0.045 0 0" rpy="0 0 0"/>
+        <origin xyz="0.025 0 0" rpy="0 0 0"/>
         <geometry>
-          <box size="0.09 0.05 0.045"/>
+          <box size="0.05 0.09 0.045"/>
         </geometry>
         <material name="dark_grey">
@@ -107,11 +107,11 @@
       </visual>
       <collision>
-        <origin xyz="0.045 0 0" rpy="0 0 0"/>
+        <origin xyz="0.025 0 0" rpy="0 0 0"/>
         <geometry>
-          <box size="0.09 0.05 0.045"/>
+          <box size="0.05 0.09 0.045"/>
         </geometry>
       </collision>
       <inertial>
-        <origin xyz="0.045 0 0" rpy="0 0 0"/>
+        <origin xyz="0.025 0 0" rpy="0 0 0"/>
         <mass value="0.02"/>
         <inertia ixx="0.00001" ixy="0.0" ixz="0.0" iyy="0.00001" iyz="0.0" izz="0.00001"/>
