Commit message: auto: update 2026-05-01 00:10:24

File: turtlebot3_manipulation/turtlebot3_manipulation_description/xacro/open_manipulator_x.urdf.xacro (robot description, xacro)
@@ -37,5 +37,5 @@
       <origin xyz="0.012 0.0 0.017" rpy="0 0 0"/>
       <axis xyz="0 0 1"/>
-      <limit velocity="4.8" effort="1" lower="${-pi*0.9}" upper="${pi*0.9}" />
+      <limit velocity="4.8" effort="1" lower="${-pi}" upper="${pi}" />
       <dynamics damping="0.1"/>
     </joint>

File: turtlebot3_simulations/turtlebot3_manipulation_gazebo/urdf/open_manipulator_x.urdf.xacro (robot description, xacro)
@@ -37,5 +37,5 @@
       <origin xyz="0.012 0.0 0.017" rpy="0 0 0"/>
       <axis xyz="0 0 1"/>
-      <limit velocity="4.8" effort="1" lower="${-pi*0.9}" upper="${pi*0.9}" />
+      <limit velocity="4.8" effort="1" lower="${-pi}" upper="${pi}" />
       <dynamics damping="0.1"/>
     </joint>

Commit message: auto: update 2026-05-17 16:35:57

File: turtlebot3_manipulation/turtlebot3_manipulation_description/xacro/open_manipulator_x.urdf.xacro (robot description, xacro)
@@ -95,5 +95,5 @@
       <parent link="${prefix}link3"/>
       <child link="${prefix}link4"/>
-      <origin xyz="0.024 0 0.128" rpy="0 0 0"/>
+      <origin xyz="0.024 0 0.128" rpy="0 1.5708 0"/>
       <axis xyz="0 1 0"/>
       <limit velocity="4.8" effort="1" lower="${-pi*0.3}" upper="${pi*0.44}" />

Commit message: auto: update 2026-05-17 16:44:24

File: turtlebot3_manipulation/turtlebot3_manipulation_description/xacro/open_manipulator_x.urdf.xacro (robot description, xacro)
@@ -95,5 +95,5 @@
       <parent link="${prefix}link3"/>
       <child link="${prefix}link4"/>
-      <origin xyz="0.024 0 0.128" rpy="0 1.5708 0"/>
+      <origin xyz="0.024 0 0.128" rpy="0 1.5708 0"/> # 영점 수정 0 -> 1.5708
       <axis xyz="0 1 0"/>
       <limit velocity="4.8" effort="1" lower="${-pi*0.3}" upper="${pi*0.44}" />

Commit message: auto: update 2026-05-17 16:44:36

File: turtlebot3_manipulation/turtlebot3_manipulation_description/xacro/open_manipulator_x.urdf.xacro (robot description, xacro)
@@ -95,5 +95,5 @@
       <parent link="${prefix}link3"/>
       <child link="${prefix}link4"/>
-      <origin xyz="0.024 0 0.128" rpy="0 1.5708 0"/> # 영점 수정 0 -> 1.5708
+      <origin xyz="0.024 0 0.128" rpy="0 1.5708 0"/> # 영점 수정 0에서 1.5708
       <axis xyz="0 1 0"/>
       <limit velocity="4.8" effort="1" lower="${-pi*0.3}" upper="${pi*0.44}" />

Commit message: auto: update 2026-05-17 16:48:53

File: turtlebot3_manipulation/turtlebot3_manipulation_description/xacro/open_manipulator_x.urdf.xacro (robot description, xacro)
@@ -95,5 +95,5 @@
       <parent link="${prefix}link3"/>
       <child link="${prefix}link4"/>
-      <origin xyz="0.024 0 0.128" rpy="0 1.5708 0"/> # 영점 수정 0에서 1.5708
+      <origin xyz="0.024 0 0.128" rpy="0 0 0"/>
       <axis xyz="0 1 0"/>
       <limit velocity="4.8" effort="1" lower="${-pi*0.3}" upper="${pi*0.44}" />
