Commit message: auto: update 2026-05-28 15:34:37

File: turtlebot3_manipulation/turtlebot3_manipulation_description/xacro/turtlebot3_platooning.xacro (robot description, xacro)
@@ -6,5 +6,5 @@
 -->
 <robot xmlns:xacro="http://www.ros.org/wiki/xacro">
-  <xacro:macro name="turtlebot3_waffle_pi" params="prefix">
+  <xacro:macro name="turtlebot3_waffle_pi" params="prefix use_collision:=true">
   <xacro:property
     name="meshes_file_direction"
@@ -24,10 +24,12 @@
       <material name="light_black"/>
     </visual>
-    <collision>
-      <origin xyz="-0.064 0 0.030" rpy="0 0 0"/>
-      <geometry>
-        <box size="0.266 0.266 0.060"/>
-      </geometry>
-    </collision>
+    <xacro:if value="${use_collision}">
+      <collision>
+        <origin xyz="-0.064 0 0.030" rpy="0 0 0"/>
+        <geometry>
+          <box size="0.266 0.266 0.060"/>
+        </geometry>
+      </collision>
+    </xacro:if>
     <inertial>
       <origin xyz="0 0 0" rpy="0 0 0"/>
@@ -52,10 +54,12 @@
       <material name="dark"/>
     </visual>
-    <collision>
-      <origin xyz="0 0 0" rpy="0 0 0"/>
-      <geometry>
-        <cylinder length="0.018" radius="0.033"/>
-      </geometry>
-    </collision>
+    <xacro:if value="${use_collision}">
+      <collision>
+        <origin xyz="0 0 0" rpy="0 0 0"/>
+        <geometry>
+          <cylinder length="0.018" radius="0.033"/>
+        </geometry>
+      </collision>
+    </xacro:if>
     <inertial>
       <origin xyz="0 0 0" />
@@ -80,10 +84,12 @@
       <material name="dark"/>
     </visual>
-    <collision>
-      <origin xyz="0 0 0" rpy="0 0 0"/>
-      <geometry>
-        <cylinder length="0.018" radius="0.033"/>
-      </geometry>
-    </collision>
+    <xacro:if value="${use_collision}">
+      <collision>
+        <origin xyz="0 0 0" rpy="0 0 0"/>
+        <geometry>
+          <cylinder length="0.018" radius="0.033"/>
+        </geometry>
+      </collision>
+    </xacro:if>
     <inertial>
       <origin xyz="0 0 0" />
@@ -100,10 +106,12 @@
   </joint>
   <link name="${prefix}caster_back_right_link">
-    <collision>
-      <origin xyz="0 0.001 0" rpy="0 0 0"/>
-      <geometry>
-        <box size="0.030 0.009 0.020"/>
-      </geometry>
-    </collision>
+    <xacro:if value="${use_collision}">
+      <collision>
+        <origin xyz="0 0.001 0" rpy="0 0 0"/>
+        <geometry>
+          <box size="0.030 0.009 0.020"/>
+        </geometry>
+      </collision>
+    </xacro:if>
     <inertial>
       <origin xyz="0 0 0" />
@@ -120,10 +128,12 @@
   </joint>
   <link name="${prefix}caster_back_left_link">
-    <collision>
-      <origin xyz="0 0.001 0" rpy="0 0 0"/>
-      <geometry>
-        <box size="0.030 0.009 0.020"/>
-      </geometry>
-    </collision>
+    <xacro:if value="${use_collision}">
+      <collision>
+        <origin xyz="0 0.001 0" rpy="0 0 0"/>
+        <geometry>
+          <box size="0.030 0.009 0.020"/>
+        </geometry>
+      </collision>
+    </xacro:if>
     <inertial>
       <origin xyz="0 0 0" />
@@ -153,10 +163,12 @@
       <material name="dark"/>
     </visual>
-    <collision>
-      <origin xyz="0 0 0" rpy="0 0 0"/>
-      <geometry>
-        <box size="0.180 0.160 0.012"/>
-      </geometry>
-    </collision>
+    <xacro:if value="${use_collision}">
+      <collision>
+        <origin xyz="0 0 0" rpy="0 0 0"/>
+        <geometry>
+          <box size="0.180 0.160 0.012"/>
+        </geometry>
+      </collision>
+    </xacro:if>
     <inertial>
       <origin xyz="0 0 0" />
@@ -173,10 +185,12 @@
   </joint>
   <link name="${prefix}camera_link">
-    <collision>
-      <origin xyz="0.005 0.011 0.013" rpy="0 0 0"/>
-      <geometry>
-        <box size="0.015 0.030 0.027"/>
-      </geometry>
-    </collision>
+    <xacro:if value="${use_collision}">
+      <collision>
+        <origin xyz="0.005 0.011 0.013" rpy="0 0 0"/>
+        <geometry>
+          <box size="0.015 0.030 0.027"/>
+        </geometry>
+      </collision>
+    </xacro:if>
   </link>
   <joint name="${prefix}camera_rgb_joint" type="fixed">

Commit message: auto: update 2026-05-28 15:47:43

File: turtlebot3_manipulation/turtlebot3_manipulation_description/xacro/turtlebot3_platooning.xacro (robot description, xacro)
@@ -6,5 +6,5 @@
 -->
 <robot xmlns:xacro="http://www.ros.org/wiki/xacro">
-  <xacro:macro name="turtlebot3_waffle_pi" params="prefix use_collision:=true">
+  <xacro:macro name="turtlebot3_waffle_pi" params="prefix">
   <xacro:property
     name="meshes_file_direction"
@@ -24,12 +24,10 @@
       <material name="light_black"/>
     </visual>
-    <xacro:if value="${use_collision}">
-      <collision>
-        <origin xyz="-0.064 0 0.030" rpy="0 0 0"/>
-        <geometry>
-          <box size="0.266 0.266 0.060"/>
-        </geometry>
-      </collision>
-    </xacro:if>
+    <collision>
+      <origin xyz="-0.064 0 0.030" rpy="0 0 0"/>
+      <geometry>
+        <box size="0.266 0.266 0.060"/>
+      </geometry>
+    </collision>
     <inertial>
       <origin xyz="0 0 0" rpy="0 0 0"/>
@@ -43,10 +41,10 @@
     <parent link="${prefix}base_link"/>
     <child link="${prefix}wheel_left_link"/>
-    <origin xyz="0.0 0.144 0.023" rpy="-1.57079632679 0 0"/>
+    <origin xyz="0.0 0.144 0.023" rpy="-1.57 0 0"/>
     <axis xyz="0 0 1"/>
   </joint>
   <link name="${prefix}wheel_left_link">
     <visual>
-      <origin xyz="0 0 0" rpy="1.57079632679 0 0"/>
+      <origin xyz="0 0 0" rpy="1.57 0 0"/>
       <geometry>
         <mesh filename="${meshes_file_direction}/left_tire.stl" scale="0.001 0.001 0.001"/>
@@ -54,12 +52,10 @@
       <material name="dark"/>
     </visual>
-    <xacro:if value="${use_collision}">
-      <collision>
-        <origin xyz="0 0 0" rpy="0 0 0"/>
-        <geometry>
-          <cylinder length="0.018" radius="0.033"/>
-        </geometry>
-      </collision>
-    </xacro:if>
+    <collision>
+      <origin xyz="0 0 0" rpy="0 0 0"/>
+      <geometry>
+        <cylinder length="0.018" radius="0.033"/>
+      </geometry>
+    </collision>
     <inertial>
       <origin xyz="0 0 0" />
@@ -73,10 +69,10 @@
     <parent link="${prefix}base_link"/>
     <child link="${prefix}wheel_right_link"/>
-    <origin xyz="0.0 -0.144 0.023" rpy="-1.57079632679 0 0"/>
+    <origin xyz="0.0 -0.144 0.023" rpy="-1.57 0 0"/>
     <axis xyz="0 0 1"/>
   </joint>
   <link name="${prefix}wheel_right_link">
     <visual>
-      <origin xyz="0 0 0" rpy="1.57079632679 0 0"/>
+      <origin xyz="0 0 0" rpy="1.57 0 0"/>
       <geometry>
         <mesh filename="${meshes_file_direction}/right_tire.stl" scale="0.001 0.001 0.001"/>
@@ -84,12 +80,10 @@
       <material name="dark"/>
     </visual>
-    <xacro:if value="${use_collision}">
-      <collision>
-        <origin xyz="0 0 0" rpy="0 0 0"/>
-        <geometry>
-          <cylinder length="0.018" radius="0.033"/>
-        </geometry>
-      </collision>
-    </xacro:if>
+    <collision>
+      <origin xyz="0 0 0" rpy="0 0 0"/>
+      <geometry>
+        <cylinder length="0.018" radius="0.033"/>
+      </geometry>
+    </collision>
     <inertial>
       <origin xyz="0 0 0" />
@@ -103,15 +97,13 @@
     <parent link="${prefix}base_link"/>
     <child link="${prefix}caster_back_right_link"/>
-    <origin xyz="-0.177 -0.064 -0.004" rpy="-1.57079632679 0 0"/>
+    <origin xyz="-0.177 -0.064 -0.004" rpy="-1.57 0 0"/>
   </joint>
   <link name="${prefix}caster_back_right_link">
-    <xacro:if value="${use_collision}">
-      <collision>
-        <origin xyz="0 0.001 0" rpy="0 0 0"/>
-        <geometry>
-          <box size="0.030 0.009 0.020"/>
-        </geometry>
-      </collision>
-    </xacro:if>
+    <collision>
+      <origin xyz="0 0.001 0" rpy="0 0 0"/>
+      <geometry>
+        <box size="0.030 0.009 0.020"/>
+      </geometry>
+    </collision>
     <inertial>
       <origin xyz="0 0 0" />
@@ -125,15 +117,13 @@
     <parent link="${prefix}base_link"/>
     <child link="${prefix}caster_back_left_link"/>
-    <origin xyz="-0.177 0.064 -0.004" rpy="-1.57079632679 0 0"/>
+    <origin xyz="-0.177 0.064 -0.004" rpy="-1.57 0 0"/>
   </joint>
   <link name="${prefix}caster_back_left_link">
-    <xacro:if value="${use_collision}">
-      <collision>
-        <origin xyz="0 0.001 0" rpy="0 0 0"/>
-        <geometry>
-          <box size="0.030 0.009 0.020"/>
-        </geometry>
-      </collision>
-    </xacro:if>
+    <collision>
+      <origin xyz="0 0.001 0" rpy="0 0 0"/>
+      <geometry>
+        <box size="0.030 0.009 0.020"/>
+      </geometry>
+    </collision>
     <inertial>
       <origin xyz="0 0 0" />
@@ -150,33 +140,4 @@
   </joint>
   <link name="${prefix}imu_link"/>
-  <joint name="${prefix}cargo_deck_joint" type="fixed">
-    <parent link="${prefix}base_link"/>
-    <child link="${prefix}cargo_deck_link"/>
-    <origin xyz="-0.045 0 0.105" rpy="0 0 0"/>
-  </joint>
-  <link name="${prefix}cargo_deck_link">
-    <visual>
-      <origin xyz="0 0 0" rpy="0 0 0"/>
-      <geometry>
-        <box size="0.180 0.160 0.012"/>
-      </geometry>
-      <material name="dark"/>
-    </visual>
-    <xacro:if value="${use_collision}">
-      <collision>
-        <origin xyz="0 0 0" rpy="0 0 0"/>
-        <geometry>
-          <box size="0.180 0.160 0.012"/>
-        </geometry>
-      </collision>
-    </xacro:if>
-    <inertial>
-      <origin xyz="0 0 0" />
-      <mass value="0.050" />
-      <inertia ixx="1.117e-04" ixy="0.0" ixz="0.0"
-               iyy="1.620e-04" iyz="0.0"
-               izz="2.417e-04" />
-    </inertial>
-  </link>
   <joint name="${prefix}camera_joint" type="fixed">
     <parent link="${prefix}base_link"/>
@@ -185,12 +146,10 @@
   </joint>
   <link name="${prefix}camera_link">
-    <xacro:if value="${use_collision}">
-      <collision>
-        <origin xyz="0.005 0.011 0.013" rpy="0 0 0"/>
-        <geometry>
-          <box size="0.015 0.030 0.027"/>
-        </geometry>
-      </collision>
-    </xacro:if>
+    <collision>
+      <origin xyz="0.005 0.011 0.013" rpy="0 0 0"/>
+      <geometry>
+        <box size="0.015 0.030 0.027"/>
+      </geometry>
+    </collision>
   </link>
   <joint name="${prefix}camera_rgb_joint" type="fixed">
@@ -203,5 +162,5 @@
     <parent link="${prefix}camera_rgb_frame"/>
     <child link="${prefix}camera_rgb_optical_frame"/>
-    <origin xyz="0 0 0" rpy="-1.57079632679 0 -1.57079632679"/>
+    <origin xyz="0 0 0" rpy="-1.57 0 -1.57"/>
   </joint>
   <link name="${prefix}camera_rgb_optical_frame"/>
