Commit message: auto: update 2026-05-08 00:49:24

File: turtlebot3_simulations/turtlebot3_manipulation_gazebo/urdf/turtlebot3_platooning_follower.urdf.xacro (robot description, xacro)
@@ -4,4 +4,4 @@
   <xacro:include filename="$(find turtlebot3_manipulation_gazebo)/gazebo/materials.xacro"/>
   <xacro:include filename="$(find turtlebot3_manipulation_gazebo)/urdf/turtlebot3_waffle_pi.urdf.xacro"/>
-  <xacro:turtlebot3_waffle_pi prefix="$(arg prefix)"/>
+  <xacro:turtlebot3_waffle_pi prefix="$(arg prefix)" wheel_joint_type="fixed"/>
 </robot>

File: turtlebot3_simulations/turtlebot3_manipulation_gazebo/urdf/turtlebot3_waffle_pi.urdf.xacro (robot description, xacro)
@@ -6,5 +6,5 @@
 -->
 <robot xmlns:xacro="http://www.ros.org/wiki/xacro">
-  <xacro:macro name="turtlebot3_waffle_pi" params="prefix">
+  <xacro:macro name="turtlebot3_waffle_pi" params="prefix wheel_joint_type:=continuous">
   <xacro:property
     name="meshes_file_direction"
@@ -38,5 +38,5 @@
     </inertial>
   </link>
-  <joint name="${prefix}wheel_left_joint" type="continuous">
+  <joint name="${prefix}wheel_left_joint" type="${wheel_joint_type}">
     <parent link="${prefix}base_link"/>
     <child link="${prefix}wheel_left_link"/>
@@ -66,5 +66,5 @@
       </inertial>
   </link>
-  <joint name="${prefix}wheel_right_joint" type="continuous">
+  <joint name="${prefix}wheel_right_joint" type="${wheel_joint_type}">
     <parent link="${prefix}base_link"/>
     <child link="${prefix}wheel_right_link"/>
